Commit message: partition(v1) tree(v2) grid size(v3) wind(v4)

File: models/iitp_drone/urdf/multirotor_base.xacro (robot description, xacro)
@@ -45,4 +45,5 @@
         <origin xyz="0 0 0" rpy="0 0 0" />
         <geometry>
+          <!-- <box size="${body_width} ${body_width} ${body_height}" /> [m] [m] [m] -->
           <box size="${body_width} ${body_width} ${body_height}" /> <!-- [m] [m] [m] -->
         </geometry>
@@ -51,4 +52,6 @@
     <!-- attach multirotor_base_plugin to the base_link -->
     <gazebo>
+      <!--this model is affected by wind  -->
+      <enable_wind>true</enable_wind>
       <plugin filename="libgazebo_multirotor_base_plugin.so" name="rosbag">
         <robotNamespace>${robot_namespace}</robotNamespace>
