Commit message: little change??

File: models/iitp_drone/urdf/component_snippets.xacro (robot description, xacro)
@@ -113,5 +113,8 @@
        <px4flow_sensor_rpy value= "$(arg px4flow_sensor_rpy)"/> -->
     <xacro:property name="px4flow_pose_rpy" value="1.57079632679 0 1.57079632679" />
-    <xacro:property name="px4flow_sensor_rpy" value="-1.57079632679 1.57079632679 0" />
+    <!-- <xacro:property name="px4flow_pose_rpy" value="0 1.57079632679 1.57079632679" /> -->
+    <!-- <xacro:property name="px4flow_sensor_rpy" value="-1.57079632679 1.57079632679 0" /> -->
+    <xacro:property name="px4flow_sensor_rpy" value="0 1.57079632679 1.5707963267" />
+    <!-- <xacro:property name="px4flow_sensor_rpy" value="0 1.57079632679 3.1415" /> -->
     </xacro:if>
     <xacro:unless value="${camera_T_sonar_F}">
@@ -160,12 +163,12 @@
           <update_rate>${frame_rate}</update_rate>
           <!-- set up visibility of beam form of camera sight> -->
-          <visualize>false</visualize>
-          <!-- <topic>/px4flow</topic> -->
+          <visualize>true</visualize>
+          <topic>/px4flow</topic>
           <camera>
             <horizontal_fov>0.25</horizontal_fov>
-            <lens>
+            <!-- <lens>
               <type>gnomonical</type>
               <scale_to_hfov>false</scale_to_hfov>
-            </lens>
+            </lens> -->
             <image>
               <width>64</width>
@@ -183,7 +186,12 @@
             </noise>
           </camera>
-          <plugin name="${namespace}_opticalflow_plugin" filename="libgazebo_opticalflow_plugin.so">
-              <robotNamespace></robotNamespace>
-              <outputRate>20</outputRate>
+          <!-- <plugin name="${namespace}_opticalflow_plugin" filename="libgazebo_opticalflow_plugin.so"> -->
+          <plugin name="px4flow" filename="libgazebo_opticalflow_plugin.so">
+              <robotNamespace>${namespace}</robotNamespace>
+              <!-- <outputRate>20</outputRate> -->
+              <updateRate>0.0</updateRate>
+              <!-- <topicName>/mavros/px4flow/raw/optical_flow_rad</topicName> -->
+              <!-- <topicName>abcdedfhijk</topicName> -->
+              <!-- <frameName>${namespace}_px4flow_${camera_T_sonar_F}_link</frameName> -->
           </plugin>
           <!-- <plugin name="${namespace}_camera_controller" filename="libgazebo_ros_camera.so">
@@ -213,9 +221,22 @@
           </sonar>
           <always_on>1</always_on>
-          <visualize>false</visualize>
-          <plugin name="${namespace}_sonar_plugin" filename="libgazebo_opticalflow_plugin.so">
+          <visualize>true</visualize>
+          <!-- <plugin name="${namespace}_sonar_plugin" filename="libgazebo_opticalflow_plugin.so">
             <robotNamespace>${namespace}</robotNamespace>
             <outputRate>20</outputRate>
+          </plugin> -->
+          <plugin name="hrlv_ez4_pub" filename="libgazebo_sonar_plugin.so">
           </plugin>
+          <!-- libgazebo_ros_range.so -->
+          <!-- <plugin name="gazebo_ros_range" filename="libgazebo_ros_range.so">
+            <robotNamespace>${namespace}</robotNamespace>
+            <gaussianNoise>0.005</gaussianNoise>
+            <alwaysOn>true</alwaysOn>
+            <updateRate>10</updateRate>
+            <topicName>sensor/hrlv_ez4_pub</topicName>
+            <frameName>${namespace}/px4flow_${camera_T_sonar_F}_link</frameName>
+            <fov>0</fov>
+            <radiation>ultrasound</radiation>
+          </plugin> -->
         </sensor>
       </xacro:unless>
@@ -255,4 +276,5 @@
       <!-- <axis xyz="0 1 0"/> -->
       <origin xyz="${lidar_xyz}" rpy="0 1.570896 0" />
+      <!-- <origin xyz="${lidar_xyz}" rpy="0 3.1415 0" /> -->
       <!-- <xacro:insert_block name="origin" /> -->
       <parent link="${parent_link}" />
@@ -261,7 +283,8 @@
     <gazebo reference="${namespace}/lidar_link">
       <sensor type="ray" name="${namespace}_lidar">
+        <!-- <pose>0 0 0 0 -1.570896 0</pose> -->
         <always_on>1</always_on>
         <update_rate>${frame_rate}</update_rate>
-        <visualize>false</visualize>
+        <visualize>true</visualize>
         <ray>
           <scan>
@@ -286,5 +309,7 @@
           </noise>
         </ray>
-        <plugin name="Laserplugin" filename="libgazebo_lidar_plugin.so">
+        <plugin name="${namespace}_Laserplugin" filename="libgazebo_lidar_plugin.so">
+        <!-- <plugin name="lidarlite_pub" filename="libgazebo_lidar_plugin.so"> -->
+          <!-- <robotNamespace>${namespace}</robotNamespace> -->
           <robotNamespace>${namespace}</robotNamespace>
           <min_distance>0.2</min_distance>

File: models/iitp_drone/urdf/iitp_drone.xacro (robot description, xacro)
@@ -58,5 +58,5 @@
   <!-- <origin xyz="0 0 -0.05" rpy="-1.57079632679 1.57079632679 0" /> -->
   <!-- add px4flow_sonar -->
-  <xacro:px4flow_macro
+  <!-- <xacro:px4flow_macro
     namespace="${namespace}"
     parent_link= "base_link"
@@ -66,6 +66,6 @@
     enable_visual="true"
     px4flow_origin_xyz="-0.025 0.05 -0.025">
-  </xacro:px4flow_macro> -->
-      <!-- frame_rate do not effect of sonar. -->
+  </xacro:px4flow_macro> --> -->
+     <!-- frame_rate do not effect of sonar. -->
     <!-- px4flow_origin_xyz="0 0 -0.08869" -->
   <!-- add lidar -->
